File: DESIGN/PCB/PowerSwitches/PowerSwitches.kicad_pcb (KiCad board)
At the start: 2 copper layers, 104.4 x 64 mm, 15 parts, among them J1 BTN REMOTE, J2 POWER OUT, J3 TEST REMOTE, SW1 ON/OFF, SW2 TEST START/STOP, U1 LV_Pushbutton_Switch, U2 HP_Pushbutton_Switch, U3 HP_Pushbutton_Switch

Commit message: Rev 1.1 of power switch pcb.
Connections:
- J1 pad 1: Net-(J1-Pad1) -> Net-(U1-Pad9)
- J3 pad 1: Net-(J3-Pad1) -> Net-(SW2-Pad3)
- SW1 pad 2: Net-(J1-Pad1) -> unconnected-(SW1-Pad2)
- SW1 pad 3: unconnected-(SW1-Pad3) -> Net-(U1-Pad9)
- SW2 pad 2: Net-(J3-Pad1) -> unconnected-(SW2-Pad2)
- SW2 pad 3: unconnected-(SW2-Pad3) -> Net-(SW2-Pad3)
- U1 pad 9: Net-(J1-Pad1) -> Net-(U1-Pad9)
Routing:
- net Net-(U1-Pad9): track 0.00 -> 29.8 mm
- net Net-(J1-Pad1): track 23.7 -> 0.00 mm
- net Net-(SW2-Pad3): track 0.00 -> 17.9 mm
- net Net-(J3-Pad1): track 11.6 -> 0.00 mm
- net Net-(J3-Pad2): track 11.8 -> 14.1 mm
- net Net-(J1-Pad2): track 29.1 -> 30.6 mm
Other:
- board text added: "POWERED SWITCHES REV 1.1"
- board text removed: "POWERED SWITCHES REV 1.0"
Changed lines of the file:
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@@
       (drillshape 0)
       (scaleselection 1)
-      (outputdirectory "REV1_0/")
+      (outputdirectory "REV1_1/")
     )
   )
@@
   (net 1 "/5V-IN")
   (net 2 "/GND-IN")
-  (net 3 "Net-(J1-Pad1)")
+  (net 3 "Net-(U1-Pad9)")
   (net 4 "Net-(J1-Pad2)")
   (net 5 "/5V-OUT")
   (net 6 "/GND-OUT")
   (net 7 "Net-(R1-Pad2)")
-  (net 8 "unconnected-(SW1-Pad3)")
+  (net 8 "Net-(SW2-Pad3)")
   (net 9 "unconnected-(SW1-Pad4)")
   (net 10 "unconnected-(U1-Pad2)")
@@
   (net 44 "unconnected-(U3-Pad16)")
   (net 45 "unconnected-(U1-Pad10)")
-  (net 46 "Net-(J3-Pad1)")
+  (net 46 "unconnected-(SW1-Pad2)")
   (net 47 "Net-(J3-Pad2)")
-  (net 48 "unconnected-(SW2-Pad3)")
+  (net 48 "unconnected-(SW2-Pad2)")
   (net 49 "unconnected-(SW2-Pad4)")
   (footprint "Custom:HV_PushButton_Switch" (layer "F.Cu")
@@
     (fp_line (start -2.45 3.4) (end 4.95 3.4) (layer "F.Fab") (width 0.1))
     (pad "1" thru_hole roundrect (at 0 0) (size 1.7 2) (drill 1) (layers *.Cu *.Mask) (roundrect_rratio 0.1470588235)
-      (net 46 "Net-(J3-Pad1)") (pinfunction "Pin_1") (pintype "passive"))
+      (net 8 "Net-(SW2-Pad3)") (pinfunction "Pin_1") (pintype "passive"))
     (pad "2" thru_hole oval (at 2.5 0) (size 1.7 2) (drill 1) (layers *.Cu *.Mask)
       (net 47 "Net-(J3-Pad2)") (pinfunction "Pin_2") (pintype "passive"))
@@
       (net 4 "Net-(J1-Pad2)") (pinfunction "A") (pintype "input"))
     (pad "9" thru_hole circle (at 5.08 2.54) (size 1.524 1.524) (drill 0.762) (layers *.Cu *.Mask)
-      (net 3 "Net-(J1-Pad1)") (pinfunction "B") (pintype "input"))
+      (net 3 "Net-(U1-Pad9)") (pinfunction "B") (pintype "input"))
     (pad "10" thru_hole circle (at 5.08 0) (size 1.524 1.524) (drill 0.762) (layers *.Cu *.Mask)
       (net 45 "unconnected-(U1-Pad10)") (pinfunction "GND") (pintype "power_out"))
@@
       (net 4 "Net-(J1-Pad2)") (pinfunction "1") (pintype "passive"))
     (pad "2" thru_hole circle (at 2.54 -2.54 180) (size 1.524 1.524) (drill 0.762) (layers *.Cu *.Mask)
-      (net 3 "Net-(J1-Pad1)") (pinfunction "2") (pintype "passive"))
+      (net 46 "unconnected-(SW1-Pad2)") (pinfunction "2") (pintype "passive"))
     (pad "3" thru_hole circle (at -5.08 2.54 180) (size 1.524 1.524) (drill 0.762) (layers *.Cu *.Mask)
-      (net 8 "unconnected-(SW1-Pad3)") (pinfunction "3") (pintype "passive"))
+      (net 3 "Net-(U1-Pad9)") (pinfunction "3") (pintype "passive"))
     (pad "4" thru_hole circle (at 2.54 2.54 180) (size 1.524 1.524) (drill 0.762) (layers *.Cu *.Mask)
       (net 9 "unconnected-(SW1-Pad4)") (pinfunction "4") (pintype "passive"))
@@
       (net 47 "Net-(J3-Pad2)") (pinfunction "1") (pintype "passive"))
     (pad "2" thru_hole circle (at 2.54 -2.54 180) (size 1.524 1.524) (drill 0.762) (layers *.Cu *.Mask)
-      (net 46 "Net-(J3-Pad1)") (pinfunction "2") (pintype "passive"))
+      (net 48 "unconnected-(SW2-Pad2)") (pinfunction "2") (pintype "passive"))
     (pad "3" thru_hole circle (at -5.08 2.54 180) (size 1.524 1.524) (drill 0.762) (layers *.Cu *.Mask)
-      (net 48 "unconnected-(SW2-Pad3)") (pinfunction "3") (pintype "passive"))
+      (net 8 "Net-(SW2-Pad3)") (pinfunction "3") (pintype "passive"))
     (pad "4" thru_hole circle (at 2.54 2.54 180) (size 1.524 1.524) (drill 0.762) (layers *.Cu *.Mask)
       (net 49 "unconnected-(SW2-Pad4)") (pinfunction "4") (pintype "passive"))
@@
     (fp_line (start -2.45 3.4) (end 4.95 3.4) (layer "F.Fab") (width 0.1))
     (pad "1" thru_hole roundrect (at 0 0) (size 1.7 2) (drill 1) (layers *.Cu *.Mask) (roundrect_rratio 0.1470588235)
-      (net 3 "Net-(J1-Pad1)") (pinfunction "Pin_1") (pintype "passive"))
+      (net 3 "Net-(U1-Pad9)") (pinfunction "Pin_1") (pintype "passive"))
     (pad "2" thru_hole oval (at 2.5 0) (size 1.7 2) (drill 1) (layers *.Cu *.Mask)
       (net 4 "Net-(J1-Pad2)") (pinfunction "Pin_2") (pintype "passive"))
@@
     (effects (font (size 1 1) (thickness 0.15)))
   )
-  (gr_text "POWERED SWITCHES\nREV 1.0" (at 103.378 46.736) (layer "F.SilkS")
+  (gr_text "POWERED SWITCHES\nREV 1.1" (at 103.378 46.736) (layer "F.SilkS")
     (effects (font (size 1 1) (thickness 0.15)) (justify left))
   )
@@
   (segment (start 147.554 72.624) (end 140.97 66.04) (width 0.25) (layer "B.Cu") (net 2))
   (segment (start 147.554 97.519) (end 147.554 72.624) (width 0.25) (layer "B.Cu") (net 2))
-  (segment (start 165.882 70.849) (end 163.322 68.289) (width 0.25) (layer "F.Cu") (net 3))
+  (segment (start 165.882 60.178) (end 170.942 55.118) (width 0.25) (layer "F.Cu") (net 3))
   (segment (start 153.67 71.12) (end 165.611 71.12) (width 0.25) (layer "F.Cu") (net 3))
-  (segment (start 163.322 68.289) (end 163.322 60.198) (width 0.25) (layer "F.Cu") (net 3))
-  (segment (start 168.382 62.758) (end 170.942 60.198) (width 0.25) (layer "F.Cu") (net 4))
+  (segment (start 165.882 70.849) (end 165.882 60.178) (width 0.25) (layer "F.Cu") (net 3))
+  (segment (start 172.72 66.294) (end 168.382 70.632) (width 0.25) (layer "F.Cu") (net 4))
+  (segment (start 168.382 70.632) (end 168.382 70.849) (width 0.25) (layer "F.Cu") (net 4))
   (segment (start 153.67 73.66) (end 168.148 73.66) (width 0.25) (layer "F.Cu") (net 4))
+  (segment (start 170.942 60.198) (end 172.72 61.976) (width 0.25) (layer "F.Cu") (net 4))
   (segment (start 168.382 73.426) (end 168.382 70.849) (width 0.25) (layer "F.Cu") (net 4))
-  (segment (start 168.382 70.849) (end 168.382 62.758) (width 0.25) (layer "F.Cu") (net 4))
+  (segment (start 172.72 61.976) (end 172.72 66.294) (width 0.25) (layer "F.Cu") (net 4))
   (segment (start 168.148 73.66) (end 168.382 73.426) (width 0.25) (layer "F.Cu") (net 4))
   (segment (start 145.034 56.388) (end 145.034 50.038) (width 0.25) (layer "F.Cu") (net 5))
@@
   (segment (start 142.748 84.328) (end 136.398 84.328) (width 0.25) (layer "F.Cu") (net 7))
   (segment (start 149.86 84.328) (end 142.748 84.328) (width 0.25) (layer "F.Cu") (net 7))
-  (segment (start 120.65 68.543) (end 120.65 60.198) (width 0.25) (layer "F.Cu") (net 46))
-  (segment (start 122.956 70.849) (end 120.65 68.543) (width 0.25) (layer "F.Cu") (net 46))
-  (segment (start 125.456 70.849) (end 125.456 63.012) (width 0.25) (layer "F.Cu") (net 47))
-  (segment (start 125.456 63.012) (end 128.27 60.198) (width 0.25) (layer "F.Cu") (net 47))
+  (segment (start 122.956 60.432) (end 128.27 55.118) (width 0.25) (layer "F.Cu") (net 8))
+  (segment (start 122.956 70.849) (end 122.956 60.432) (width 0.25) (layer "F.Cu") (net 8))
+  (segment (start 130.81 65.786) (end 125.747 70.849) (width 0.25) (layer "F.Cu") (net 47))
+  (segment (start 128.27 60.198) (end 130.81 62.738) (width 0.25) (layer "F.Cu") (net 47))
+  (segment (start 130.81 62.738) (end 130.81 65.786) (width 0.25) (layer "F.Cu") (net 47))
+  (segment (start 125.747 70.849) (end 125.456 70.849) (width 0.25) (layer "F.Cu") (net 47))
   (zone (net 2) (net_name "/GND-IN") (layer "F.Cu") (hatch edge 0.508)
     (connect_pads (clearance 0.508))
