File: DESIGN/PCB/PowerSwitches/PowerSwitches.kicad_sch (KiCad schematic)
At the start: 11 parts, among them J1 BTN REMOTE, J2 POWER OUT, J3 TEST REMOTE, SW1 ON/OFF, SW2 TEST START/STOP, U1 LV_Pushbutton_Switch, U2 HP_Pushbutton_Switch, U3 HP_Pushbutton_Switch

Commit message: Rev 1.1 of power switch pcb.
Connections:
- net at J1.1 (Pin_1), U1.9 (B): now also SW1.3; no longer SW1.2
- net at SW2.2: no longer J3.1 (Pin_1)
- net at SW2.3: now also J3.1 (Pin_1)
Changed lines of the file:
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@@
 (kicad_sch (version 20211123) (generator eeschema)
   (paper "A4")
+  (junction (at 113.03 97.79) (diameter 0) (color 0 0 0 0)
+  )
   (junction (at 142.24 92.71) (diameter 0) (color 0 0 0 0)
   )
   (junction (at 91.44 87.63) (diameter 0) (color 0 0 0 0)
   )
-  (junction (at 113.03 87.63) (diameter 0) (color 0 0 0 0)
-  )
   (junction (at 142.24 121.92) (diameter 0) (color 0 0 0 0)
   )
   (junction (at 77.47 46.99) (diameter 0) (color 0 0 0 0)
+  )
+  (wire (pts (xy 93.98 92.71) (xy 97.79 92.71))
+    (stroke (width 0) (type default) (color 0 0 0 0))
   )
   (wire (pts (xy 77.47 46.99) (xy 77.47 63.5))
@@
     (stroke (width 0) (type default) (color 0 0 0 0))
   )
-  (wire (pts (xy 121.92 87.63) (xy 113.03 87.63))
-    (stroke (width 0) (type default) (color 0 0 0 0))
-  )
   (wire (pts (xy 116.84 71.12) (xy 119.38 71.12))
     (stroke (width 0) (type default) (color 0 0 0 0))
   )
-  (wire (pts (xy 91.44 102.87) (xy 101.6 102.87))
+  (wire (pts (xy 113.03 97.79) (xy 113.03 102.87))
     (stroke (width 0) (type default) (color 0 0 0 0))
   )
-  (wire (pts (xy 213.36 82.55) (xy 220.98 82.55))
+  (wire (pts (xy 91.44 102.87) (xy 101.6 102.87))
     (stroke (width 0) (type default) (color 0 0 0 0))
   )
@@
     (stroke (width 0) (type default) (color 0 0 0 0))
   )
+  (wire (pts (xy 205.74 76.2) (xy 205.74 72.39))
+    (stroke (width 0) (type default) (color 0 0 0 0))
+  )
   (wire (pts (xy 116.84 58.42) (xy 143.51 58.42))
     (stroke (width 0) (type default) (color 0 0 0 0))
   )
-  (wire (pts (xy 113.03 87.63) (xy 107.95 87.63))
+  (wire (pts (xy 113.03 97.79) (xy 93.98 97.79))
+    (stroke (width 0) (type default) (color 0 0 0 0))
+  )
+  (wire (pts (xy 121.92 87.63) (xy 113.03 87.63))
     (stroke (width 0) (type default) (color 0 0 0 0))
   )
@@
     (stroke (width 0) (type default) (color 0 0 0 0))
   )
-  (wire (pts (xy 220.98 82.55) (xy 220.98 67.31))
+  (wire (pts (xy 113.03 87.63) (xy 113.03 97.79))
     (stroke (width 0) (type default) (color 0 0 0 0))
   )
@@
     (stroke (width 0) (type default) (color 0 0 0 0))
   )
+  (wire (pts (xy 205.74 72.39) (xy 207.01 72.39))
+    (stroke (width 0) (type default) (color 0 0 0 0))
+  )
   (wire (pts (xy 91.44 78.74) (xy 91.44 87.63))
+    (stroke (width 0) (type default) (color 0 0 0 0))
+  )
+  (wire (pts (xy 213.36 82.55) (xy 213.36 76.2))
     (stroke (width 0) (type default) (color 0 0 0 0))
   )
@@
     (stroke (width 0) (type default) (color 0 0 0 0))
   )
-  (wire (pts (xy 217.17 67.31) (xy 220.98 67.31))
+  (wire (pts (xy 213.36 76.2) (xy 205.74 76.2))
     (stroke (width 0) (type default) (color 0 0 0 0))
   )
@@
     (stroke (width 0) (type default) (color 0 0 0 0))
   )
-  (wire (pts (xy 113.03 87.63) (xy 113.03 102.87))
-    (stroke (width 0) (type default) (color 0 0 0 0))
-  )
   (wire (pts (xy 77.47 63.5) (xy 101.6 63.5))
     (stroke (width 0) (type default) (color 0 0 0 0))
   )
+  (wire (pts (xy 93.98 97.79) (xy 93.98 92.71))
+    (stroke (width 0) (type default) (color 0 0 0 0))
+  )
